Commit message: minor updates - imu working well

File: urdf/zumobot.urdf (robot description, URDF)
Before this commit: robot zumobot, 5 links, 4 joints
Links:
- added link base_footprint; visual box size=0.001 0.001 0.001
Joints:
- added joint footprint_base_joint: type fixed, parent base_footprint, child base_link, origin xyz=0 0 0.027
- joint pan_joint: origin xyz=0 0 0.05 -> xyz=0 0 0.023
